File: mv2/mv2.kicad_sch (KiCad schematic)
At the start: 49 parts, among them J1 SWD, J2 Conn_01x04, J3 USB_C_Receptacle_USB2.0, SW1 SW_Push, U1 RP2040, U2 USBLC6-2SC6, U3 W25Q128JVS, Y1 12MHz

Commit message: pcb routed
Parts:
- removed R10, R4, R5, R6, R7, R8, R9: R_Small, symbol Device:R_Small
- removed R2, R3: 27R, Resistor_SMD:R_0603_1608Metric, symbol Device:R_Small
- removed S1, S2, S3, S4, S5, S6, S7, S8, S9: keys, CHERRY-MX-LED, symbol SparkFun-Switches:MOMENTARY-SWITCH-SPST-LED-PTH-CHERRY
- removed U1: RP2040, Sleep-Lib:RP2040-QFN-56, symbol Sleep-lib:RP2040
- added C1, C3: 1uF, Capacitor_SMD:C_0402_1005Metric, symbol Device:C_Small
- added SW1: RotaryEncoder_Switch, symbol Device:RotaryEncoder_Switch
- added U1, U10, U11, U12, U13, U2, U3, U4, U6, U7, U8, U9: MX1A-11NN, CHERRY_MX1A-11NN_SWITCH, symbol MX1A-11NN:MX1A-11NN
- added U14: XC6206PxxxMR-Regulator_Linear, Package_TO_SOT_SMD:SOT-23, symbol kicad-keyboard-parts:XC6206PxxxMR-Regulator_Linear
- added U5: RP2040, QFN40P700X700X90-57N, symbol RP2040:RP2040
- R11, R12: value R_Small -> 27R; footprint (none) -> Resistor_SMD:R_0603_1608Metric; LCSC (none) -> C25190
- renumbered C8 to C10, C9 to C11, C10 to C12, C11 to C13, C12 to C14, C13 to C15, C14 to C16, C15 to C17, C1 to C2, C2 to C4, C3 to C5, C4 to C6, C5 to C7, C6 to C8, C7 to C9, R13 to R17, R14 to R18, R15 to R19, R16 to R20, SW1 to SW2, U2 to U15, U3 to U16
Connections:
- net +1V1: now also U5.23 (DVDD), U5.45 (VREG_VOUT), U5.50 (DVDD)
- net +3V3: now also C3.2, U14.2 (VO), U5.1 (IOVDD), U5.10 (IOVDD), U5.22 (IOVDD), U5.33 (IOVDD), U5.42 (IOVDD), U5.43 (ADC_AVDD), U5.44 (VREG_VIN), U5.48 (USB_VDD), U5.49 (IOVDD)
- net +5V: now also C1.2, U14.3 (VI)
- net But_1: now also U2.P$1, U5.3 (GPIO1)
- net But_2: now also U5.4 (GPIO2), U9.P$1
- net But_3: now also U12.P$1, U5.5 (GPIO3)
- net But_4: now also U3.P$1, U5.6 (GPIO4)
- net But_5: now also U5.7 (GPIO5), U7.P$1
- net But_6: now also U10.P$1, U5.8 (GPIO6)
- net But_7: now also U4.P$1, U5.9 (GPIO7)
- net But_8: now also U5.11 (GPIO8), U8.P$1
- net But_9: now also U13.P$1, U5.12 (GPIO9)
- net CS: now also U5.56 (QSPI_CSN)
- net D_N: now also R11.1
- net D_P: now also R12.1
- net GND: now also C1.1, C3.1, U1.P$2, U10.P$2, U11.P$2, U12.P$2, U13.P$2, U14.1 (GND), U2.P$2, U3.P$2, U4.P$2, U5.19 (TESTEN), U5.57 (GND), U6.P$2, U7.P$2, U8.P$2, U9.P$2; no longer R11.2, R12.2
- net GPI0 17: now also U5.28 (GPIO17)
- net GPIO 18: now also U5.29 (GPIO18)
- net QSPI_CLK: now also U5.52 (QSPI_SCLK)
- net SD0: now also U5.53 (QSPI_SD0)
- net SD1: now also U5.55 (QSPI_SD1)
- net SD2: now also U5.54 (QSPI_SD2)
- net SD3: now also U5.51 (QSPI_SD3)
- net SWCLK: now also U5.24 (SWCLK)
- net SWD: now also U5.25 (SWD)
- net XTAL_IN: now also U5.20 (XIN)
- net XTAL_OUT: now also U5.21 (XOUT)
- new net: R12.2, U5.47 (USB_DP)
- new net: R11.2, U5.46 (USB_DM)
- new net But_10: U1.P$1, U5.35 (GPIO23)
- new net But_11: U5.14 (GPIO11), U6.P$1
- new net But_12: U11.P$1, U5.15 (GPIO12)
